File: eps/Telem.sch (KiCad schematic (older format))
At the start: 56 parts, among them Q28 IRLML6344, Q29 IRLML6344, Q30 IRLML6344, Q31 IRLML6344, Q32 IRLML6344, Q33 IRLML6344, Q34 IRLML6344, Q35 IRLML6344, Q36 IRLML6344, Q37 IRLML6344, Q38 IRLML6344, Q39 IRLML6344, Q40 IRLML6344, Q41 IRLML6344, Q42 IRLML6344, U27 CD74HC4067M, U28 74HC595, U29 74HC595, U4 CD74HC4067M

Commit message: update pcbnew
Parts:
- C24, C25, C30, C31: footprint (none) -> Capacitor_SMD:C_0805_2012Metric_Pad1.18x1.45mm_HandSolder
- R100, R101, R102, R103, R104, R105, R106, R107, R108, R109, R110, R111, R112, R113, R114, R115, R116, R117, R118, R119, R120, R121, R122, R123, R124, R91, R95, R96, R97, R98, R99: footprint (none) -> Resistor_SMD:R_0805_2012Metric_Pad1.20x1.40mm_HandSolder
- U28, U29: footprint (none) -> Package_SO:SO-16_3.9x9.9mm_P1.27mm
Changed lines of the file:
@@
 F 0 "R91" H 4370 2296 50  0000 L CNN
 F 1 "100K" H 4370 2205 50  0000 L CNN
-F 2 "" V 4230 2250 50  0001 C CNN
+F 2 "Resistor_SMD:R_0805_2012Metric_Pad1.20x1.40mm_HandSolder" V 4230 2250 50  0001 C CNN
 F 3 "~" H 4300 2250 50  0001 C CNN
 	1    4300 2250
@@
 F 0 "C25" H 2015 1146 50  0000 L CNN
 F 1 "0.1uF" H 2015 1055 50  0000 L CNN
-F 2 "" H 1938 950 50  0001 C CNN
+F 2 "Capacitor_SMD:C_0805_2012Metric_Pad1.18x1.45mm_HandSolder" H 1938 950 50  0001 C CNN
 F 3 "~" H 1900 1100 50  0001 C CNN
 	1    1900 1100
@@
 F 0 "C24" H 2015 3896 50  0000 L CNN
 F 1 "0.1uF" H 2015 3805 50  0000 L CNN
-F 2 "" H 1938 3700 50  0001 C CNN
+F 2 "Capacitor_SMD:C_0805_2012Metric_Pad1.18x1.45mm_HandSolder" H 1938 3700 50  0001 C CNN
 F 3 "~" H 1900 3850 50  0001 C CNN
 	1    1900 3850
@@
 F 0 "R96" H 4750 4100 50  0000 L CNN
 F 1 "1K" H 4750 4000 50  0000 L CNN
-F 2 "" H 4900 4050 50  0001 C CNN
+F 2 "Resistor_SMD:R_0805_2012Metric_Pad1.20x1.40mm_HandSolder" H 4900 4050 50  0001 C CNN
 F 3 "~" H 4900 4050 50  0001 C CNN
 	1    4900 4050
@@
 F 0 "R95" H 4750 3900 50  0000 L CNN
 F 1 "2.7K" H 4700 3800 50  0000 L CNN
-F 2 "" H 4900 3850 50  0001 C CNN
+F 2 "Resistor_SMD:R_0805_2012Metric_Pad1.20x1.40mm_HandSolder" H 4900 3850 50  0001 C CNN
 F 3 "~" H 4900 3850 50  0001 C CNN
 	1    4900 3850
@@
 F 0 "R98" H 5600 4100 50  0000 L CNN
 F 1 "1K" H 5600 4000 50  0000 L CNN
-F 2 "" H 5750 4050 50  0001 C CNN
+F 2 "Resistor_SMD:R_0805_2012Metric_Pad1.20x1.40mm_HandSolder" H 5750 4050 50  0001 C CNN
 F 3 "~" H 5750 4050 50  0001 C CNN
 	1    5750 4050
@@
 F 0 "R97" H 5600 3900 50  0000 L CNN
 F 1 "3.9K" H 5550 3800 50  0000 L CNN
-F 2 "" H 5750 3850 50  0001 C CNN
+F 2 "Resistor_SMD:R_0805_2012Metric_Pad1.20x1.40mm_HandSolder" H 5750 3850 50  0001 C CNN
 F 3 "~" H 5750 3850 50  0001 C CNN
 	1    5750 3850
@@
 F 0 "R100" H 6450 4100 50  0000 L CNN
 F 1 "1K" H 6450 4000 50  0000 L CNN
-F 2 "" H 6600 4050 50  0001 C CNN
+F 2 "Resistor_SMD:R_0805_2012Metric_Pad1.20x1.40mm_HandSolder" H 6600 4050 50  0001 C CNN
 F 3 "~" H 6600 4050 50  0001 C CNN
 	1    6600 4050
@@
 F 0 "R99" H 6450 3900 50  0000 L CNN
 F 1 "2.7K" H 6400 3800 50  0000 L CNN
-F 2 "" H 6600 3850 50  0001 C CNN
+F 2 "Resistor_SMD:R_0805_2012Metric_Pad1.20x1.40mm_HandSolder" H 6600 3850 50  0001 C CNN
 F 3 "~" H 6600 3850 50  0001 C CNN
 	1    6600 3850
@@
 F 0 "R102" H 7300 4100 50  0000 L CNN
 F 1 "1K" H 7300 4000 50  0000 L CNN
-F 2 "" H 7450 4050 50  0001 C CNN
+F 2 "Resistor_SMD:R_0805_2012Metric_Pad1.20x1.40mm_HandSolder" H 7450 4050 50  0001 C CNN
 F 3 "~" H 7450 4050 50  0001 C CNN
 	1    7450 4050
@@
 F 0 "R101" H 7300 3900 50  0000 L CNN
 F 1 "1.2K" H 7250 3800 50  0000 L CNN
-F 2 "" H 7450 3850 50  0001 C CNN
+F 2 "Resistor_SMD:R_0805_2012Metric_Pad1.20x1.40mm_HandSolder" H 7450 3850 50  0001 C CNN
 F 3 "~" H 7450 3850 50  0001 C CNN
 	1    7450 3850
@@
 F 0 "R104" H 8150 4100 50  0000 L CNN
 F 1 "1K" H 8150 4000 50  0000 L CNN
-F 2 "" H 8300 4050 50  0001 C CNN
+F 2 "Resistor_SMD:R_0805_2012Metric_Pad1.20x1.40mm_HandSolder" H 8300 4050 50  0001 C CNN
 F 3 "~" H 8300 4050 50  0001 C CNN
 	1    8300 4050
@@
 F 0 "R103" H 8150 3900 50  0000 L CNN
 F 1 "1.2K" H 8100 3800 50  0000 L CNN
-F 2 "" H 8300 3850 50  0001 C CNN
+F 2 "Resistor_SMD:R_0805_2012Metric_Pad1.20x1.40mm_HandSolder" H 8300 3850 50  0001 C CNN
 F 3 "~" H 8300 3850 50  0001 C CNN
 	1    8300 3850
@@
 F 0 "R106" H 9000 4100 50  0000 L CNN
 F 1 "1K" H 9000 4000 50  0000 L CNN
-F 2 "" H 9150 4050 50  0001 C CNN
+F 2 "Resistor_SMD:R_0805_2012Metric_Pad1.20x1.40mm_HandSolder" H 9150 4050 50  0001 C CNN
 F 3 "~" H 9150 4050 50  0001 C CNN
 	1    9150 4050
@@
 F 0 "R105" H 9000 3900 50  0000 L CNN
 F 1 "3.9K" H 8950 3800 50  0000 L CNN
-F 2 "" H 9150 3850 50  0001 C CNN
+F 2 "Resistor_SMD:R_0805_2012Metric_Pad1.20x1.40mm_HandSolder" H 9150 3850 50  0001 C CNN
 F 3 "~" H 9150 3850 50  0001 C CNN
 	1    9150 3850
@@
 F 0 "R108" H 9850 4100 50  0000 L CNN
 F 1 "1K" H 9850 4000 50  0000 L CNN
-F 2 "" H 10000 4050 50  0001 C CNN
+F 2 "Resistor_SMD:R_0805_2012Metric_Pad1.20x1.40mm_HandSolder" H 10000 4050 50  0001 C CNN
 F 3 "~" H 10000 4050 50  0001 C CNN
 	1    10000 4050
@@
 F 0 "R107" H 9850 3900 50  0000 L CNN
 F 1 "3.9K" H 9800 3800 50  0000 L CNN
-F 2 "" H 10000 3850 50  0001 C CNN
+F 2 "Resistor_SMD:R_0805_2012Metric_Pad1.20x1.40mm_HandSolder" H 10000 3850 50  0001 C CNN
 F 3 "~" H 10000 3850 50  0001 C CNN
 	1    10000 3850
@@
 F 0 "R110" H 10700 4100 50  0000 L CNN
 F 1 "1K" H 10700 4000 50  0000 L CNN
-F 2 "" H 10850 4050 50  0001 C CNN
+F 2 "Resistor_SMD:R_0805_2012Metric_Pad1.20x1.40mm_HandSolder" H 10850 4050 50  0001 C CNN
 F 3 "~" H 10850 4050 50  0001 C CNN
 	1    10850 4050
@@
 F 0 "R109" H 10700 3900 50  0000 L CNN
 F 1 "2.7K" H 10650 3800 50  0000 L CNN
-F 2 "" H 10850 3850 50  0001 C CNN
+F 2 "Resistor_SMD:R_0805_2012Metric_Pad1.20x1.40mm_HandSolder" H 10850 3850 50  0001 C CNN
 F 3 "~" H 10850 3850 50  0001 C CNN
 	1    10850 3850
@@
 F 0 "R112" H 4750 5400 50  0000 L CNN
 F 1 "1K" H 4750 5300 50  0000 L CNN
-F 2 "" H 4900 5350 50  0001 C CNN
+F 2 "Resistor_SMD:R_0805_2012Metric_Pad1.20x1.40mm_HandSolder" H 4900 5350 50  0001 C CNN
 F 3 "~" H 4900 5350 50  0001 C CNN
 	1    4900 5350
@@
 F 0 "R111" H 4750 5200 50  0000 L CNN
 F 1 "2.7K" H 4700 5100 50  0000 L CNN
-F 2 "" H 4900 5150 50  0001 C CNN
+F 2 "Resistor_SMD:R_0805_2012Metric_Pad1.20x1.40mm_HandSolder" H 4900 5150 50  0001 C CNN
 F 3 "~" H 4900 5150 50  0001 C CNN
 	1    4900 5150
@@
 F 0 "R114" H 5600 5400 50  0000 L CNN
 F 1 "1K" H 5600 5300 50  0000 L CNN
-F 2 "" H 5750 5350 50  0001 C CNN
+F 2 "Resistor_SMD:R_0805_2012Metric_Pad1.20x1.40mm_HandSolder" H 5750 5350 50  0001 C CNN
 F 3 "~" H 5750 5350 50  0001 C CNN
 	1    5750 5350
@@
 F 0 "R113" H 5600 5200 50  0000 L CNN
 F 1 "1.2K" H 5550 5100 50  0000 L CNN
-F 2 "" H 5750 5150 50  0001 C CNN
+F 2 "Resistor_SMD:R_0805_2012Metric_Pad1.20x1.40mm_HandSolder" H 5750 5150 50  0001 C CNN
 F 3 "~" H 5750 5150 50  0001 C CNN
 	1    5750 5150
@@
 F 0 "R116" H 6450 5400 50  0000 L CNN
 F 1 "1K" H 6450 5300 50  0000 L CNN
-F 2 "" H 6600 5350 50  0001 C CNN
+F 2 "Resistor_SMD:R_0805_2012Metric_Pad1.20x1.40mm_HandSolder" H 6600 5350 50  0001 C CNN
 F 3 "~" H 6600 5350 50  0001 C CNN
 	1    6600 5350
@@
 F 0 "R115" H 6450 5200 50  0000 L CNN
 F 1 "1.2K" H 6400 5100 50  0000 L CNN
-F 2 "" H 6600 5150 50  0001 C CNN
+F 2 "Resistor_SMD:R_0805_2012Metric_Pad1.20x1.40mm_HandSolder" H 6600 5150 50  0001 C CNN
 F 3 "~" H 6600 5150 50  0001 C CNN
 	1    6600 5150
@@
 F 0 "R118" H 7300 5400 50  0000 L CNN
 F 1 "1K" H 7300 5300 50  0000 L CNN
-F 2 "" H 7450 5350 50  0001 C CNN
+F 2 "Resistor_SMD:R_0805_2012Metric_Pad1.20x1.40mm_HandSolder" H 7450 5350 50  0001 C CNN
 F 3 "~" H 7450 5350 50  0001 C CNN
 	1    7450 5350
@@
 F 0 "R117" H 7300 5200 50  0000 L CNN
 F 1 "1.2K" H 7250 5100 50  0000 L CNN
-F 2 "" H 7450 5150 50  0001 C CNN
+F 2 "Resistor_SMD:R_0805_2012Metric_Pad1.20x1.40mm_HandSolder" H 7450 5150 50  0001 C CNN
 F 3 "~" H 7450 5150 50  0001 C CNN
 	1    7450 5150
@@
 F 0 "R120" H 8150 5400 50  0000 L CNN
 F 1 "1K" H 8150 5300 50  0000 L CNN
-F 2 "" H 8300 5350 50  0001 C CNN
+F 2 "Resistor_SMD:R_0805_2012Metric_Pad1.20x1.40mm_HandSolder" H 8300 5350 50  0001 C CNN
 F 3 "~" H 8300 5350 50  0001 C CNN
 	1    8300 5350
@@
 F 0 "R119" H 8150 5200 50  0000 L CNN
 F 1 "1.2K" H 8100 5100 50  0000 L CNN
-F 2 "" H 8300 5150 50  0001 C CNN
+F 2 "Resistor_SMD:R_0805_2012Metric_Pad1.20x1.40mm_HandSolder" H 8300 5150 50  0001 C CNN
 F 3 "~" H 8300 5150 50  0001 C CNN
 	1    8300 5150
@@
 F 0 "R122" H 9000 5400 50  0000 L CNN
 F 1 "1K" H 9000 5300 50  0000 L CNN
-F 2 "" H 9150 5350 50  0001 C CNN
+F 2 "Resistor_SMD:R_0805_2012Metric_Pad1.20x1.40mm_HandSolder" H 9150 5350 50  0001 C CNN
 F 3 "~" H 9150 5350 50  0001 C CNN
 	1    9150 5350
@@
 F 0 "R121" H 9000 5200 50  0000 L CNN
 F 1 "1.2K" H 8950 5100 50  0000 L CNN
-F 2 "" H 9150 5150 50  0001 C CNN
+F 2 "Resistor_SMD:R_0805_2012Metric_Pad1.20x1.40mm_HandSolder" H 9150 5150 50  0001 C CNN
 F 3 "~" H 9150 5150 50  0001 C CNN
 	1    9150 5150
@@
 F 0 "R124" H 9850 5400 50  0000 L CNN
 F 1 "1K" H 9850 5300 50  0000 L CNN
-F 2 "" H 10000 5350 50  0001 C CNN
+F 2 "Resistor_SMD:R_0805_2012Metric_Pad1.20x1.40mm_HandSolder" H 10000 5350 50  0001 C CNN
 F 3 "~" H 10000 5350 50  0001 C CNN
 	1    10000 5350
@@
 F 0 "R123" H 9850 5200 50  0000 L CNN
 F 1 "1.2K" H 9800 5100 50  0000 L CNN
-F 2 "" H 10000 5150 50  0001 C CNN
+F 2 "Resistor_SMD:R_0805_2012Metric_Pad1.20x1.40mm_HandSolder" H 10000 5150 50  0001 C CNN
 F 3 "~" H 10000 5150 50  0001 C CNN
 	1    10000 5150
@@
 F 0 "U28" H 8000 3181 50  0000 C CNN
 F 1 "74HC595" H 8000 3090 50  0000 C CNN
-F 2 "" H 8000 2400 50  0001 C CNN
+F 2 "Package_SO:SO-16_3.9x9.9mm_P1.27mm" H 8000 2400 50  0001 C CNN
 F 3 "http://www.ti.com/lit/ds/symlink/sn74hc595.pdf" H 8000 2400 50  0001 C CNN
 	1    8000 2400
@@
 F 0 "U29" H 9400 3181 50  0000 C CNN
 F 1 "74HC595" H 9400 3090 50  0000 C CNN
-F 2 "" H 9400 2400 50  0001 C CNN
+F 2 "Package_SO:SO-16_3.9x9.9mm_P1.27mm" H 9400 2400 50  0001 C CNN
 F 3 "http://www.ti.com/lit/ds/symlink/sn74hc595.pdf" H 9400 2400 50  0001 C CNN
 	1    9400 2400
@@
 F 0 "C30" H 7065 1996 50  0000 L CNN
 F 1 "0.1uF" H 7065 1905 50  0000 L CNN
-F 2 "" H 6988 1800 50  0001 C CNN
+F 2 "Capacitor_SMD:C_0805_2012Metric_Pad1.18x1.45mm_HandSolder" H 6988 1800 50  0001 C CNN
 F 3 "~" H 6950 1950 50  0001 C CNN
 	1    6950 1950
@@
 F 0 "C31" H 10265 1996 50  0000 L CNN
 F 1 "0.1uF" H 10265 1905 50  0000 L CNN
-F 2 "" H 10188 1800 50  0001 C CNN
+F 2 "Capacitor_SMD:C_0805_2012Metric_Pad1.18x1.45mm_HandSolder" H 10188 1800 50  0001 C CNN
 F 3 "~" H 10150 1950 50  0001 C CNN
 	1    10150 1950
