File: eps/eps.sch (KiCad schematic (older format))
At the start: 13 parts, among them Q43 IRF7425, U22 STM32F103C8Tx, U24 MAX6369

Commit message: update pcbnew
Parts:
- C23, C26, C27, C28, C29: footprint (none) -> Capacitor_SMD:C_0805_2012Metric_Pad1.18x1.45mm_HandSolder
- H1, H2: footprint (none) -> Connector_PinSocket_2.54mm:PinSocket_2x26_P2.54mm_Vertical
- R92, R93, R94: footprint (none) -> Resistor_SMD:R_0805_2012Metric_Pad1.20x1.40mm_HandSolder
Changed lines of the file:
@@
 F 0 "H1" H 1000 4267 50  0000 C CNN
 F 1 "EPS Stack Header 2" H 1000 4176 50  0000 C CNN
-F 2 "" H 950 2850 50  0001 C CNN
+F 2 "Connector_PinSocket_2.54mm:PinSocket_2x26_P2.54mm_Vertical" H 950 2850 50  0001 C CNN
 F 3 "~" H 950 2850 50  0001 C CNN
 	1    950  2850
@@
 F 0 "H2" H 2500 4267 50  0000 C CNN
 F 1 "EPS Stack Header 1" H 2500 4176 50  0000 C CNN
-F 2 "" H 2450 2850 50  0001 C CNN
+F 2 "Connector_PinSocket_2.54mm:PinSocket_2x26_P2.54mm_Vertical" H 2450 2850 50  0001 C CNN
 F 3 "~" H 2450 2850 50  0001 C CNN
 	1    2450 2850
@@
 F 0 "R94" H 8350 1450 50  0000 L CNN
 F 1 "10K" V 8300 1350 50  0000 L CNN
-F 2 "" V 8230 1450 50  0001 C CNN
+F 2 "Resistor_SMD:R_0805_2012Metric_Pad1.20x1.40mm_HandSolder" V 8230 1450 50  0001 C CNN
 F 3 "~" H 8300 1450 50  0001 C CNN
 	1    8300 1450
@@
 F 0 "R92" H 6900 1650 50  0000 L CNN
 F 1 "10K" V 6850 1550 50  0000 L CNN
-F 2 "" V 6780 1650 50  0001 C CNN
+F 2 "Resistor_SMD:R_0805_2012Metric_Pad1.20x1.40mm_HandSolder" V 6780 1650 50  0001 C CNN
 F 3 "~" H 6850 1650 50  0001 C CNN
 	1    6850 1650
@@
 F 0 "R93" H 7200 2200 50  0000 L CNN
 F 1 "50K" V 7150 2100 50  0000 L CNN
-F 2 "" V 7080 2200 50  0001 C CNN
+F 2 "Resistor_SMD:R_0805_2012Metric_Pad1.20x1.40mm_HandSolder" V 7080 2200 50  0001 C CNN
 F 3 "~" H 7150 2200 50  0001 C CNN
 	1    7150 2200
@@
 F 0 "C23" H 6865 2246 50  0000 L CNN
 F 1 "0.1uF" H 6865 2155 50  0000 L CNN
-F 2 "" H 6788 2050 50  0001 C CNN
+F 2 "Capacitor_SMD:C_0805_2012Metric_Pad1.18x1.45mm_HandSolder" H 6788 2050 50  0001 C CNN
 F 3 "~" H 6750 2200 50  0001 C CNN
 	1    6750 2200
@@
 F 0 "C29" H 10515 1196 50  0000 L CNN
 F 1 "1uF" H 10515 1105 50  0000 L CNN
-F 2 "" H 10438 1000 50  0001 C CNN
+F 2 "Capacitor_SMD:C_0805_2012Metric_Pad1.18x1.45mm_HandSolder" H 10438 1000 50  0001 C CNN
 F 3 "~" H 10400 1150 50  0001 C CNN
 	1    10400 1150
@@
 F 0 "C28" H 10065 1196 50  0000 L CNN
 F 1 "0.1uF" H 10065 1105 50  0000 L CNN
-F 2 "" H 9988 1000 50  0001 C CNN
+F 2 "Capacitor_SMD:C_0805_2012Metric_Pad1.18x1.45mm_HandSolder" H 9988 1000 50  0001 C CNN
 F 3 "~" H 9950 1150 50  0001 C CNN
 	1    9950 1150
@@
 F 0 "C27" H 8215 3496 50  0000 L CNN
 F 1 "1uF" H 8215 3405 50  0000 L CNN
-F 2 "" H 8138 3300 50  0001 C CNN
+F 2 "Capacitor_SMD:C_0805_2012Metric_Pad1.18x1.45mm_HandSolder" H 8138 3300 50  0001 C CNN
 F 3 "~" H 8100 3450 50  0001 C CNN
 	1    8100 3450
@@
 F 0 "C26" H 7765 3496 50  0000 L CNN
 F 1 "0.1uF" H 7765 3405 50  0000 L CNN
-F 2 "" H 7688 3300 50  0001 C CNN
+F 2 "Capacitor_SMD:C_0805_2012Metric_Pad1.18x1.45mm_HandSolder" H 7688 3300 50  0001 C CNN
 F 3 "~" H 7650 3450 50  0001 C CNN
 	1    7650 3450
